File: proyecto y diseño electornico/medidor de conductividad/medidor de conductividad.kicad_sch (KiCad schematic)
At the start: 44 parts, among them J1 HEADER_2, J4 Cable_PAD, U1 CD4060BM, U2 TL084, U3 LM317, U4 TC7660

Commit message: 6/5
Parts:
- C1, C2, C4, C6, C7: footprint (none) -> EESTN5:CAP_0.1
- C10, C11, C12, C13, C14, C3, C5, C9: footprint (none) -> EESTN5:CAP_ELEC_5x11mm
- C8: value (none) -> 1u; footprint (none) -> EESTN5:CAP_ELEC_5x11mm
- D1, D2, D3: footprint (none) -> EESTN5:DO-41
- D4: value (none) -> 1N5819W; footprint (none) -> EESTN5:DO-41
- D5: value (none) -> 1N4148; footprint (none) -> EESTN5:DO-41
- J1: footprint (none) -> EESTN5:BORNERA2_AZUL
- J2, J3: value (none) -> Cable_PAD; footprint (none) -> EESTN5:Cable_Doble_1,5mm
- J4: footprint (none) -> EESTN5:Cable_Doble_1,5mm
- J5: value (none) -> CONN_01X03; footprint (none) -> EESTN5:BORNERA3
- LED1: value (none) -> LED; footprint (none) -> EESTN5:led_3mm_red
- R1, R11, R14, R15, R2, R3, R4, R5, R6, R8: footprint (none) -> EESTN5:RES0.3
- R10, R12, R7, R9: value (none) -> 10k; footprint (none) -> EESTN5:RES0.3
- R13: value (none) -> 5.6k; footprint (none) -> EESTN5:RES0.3
- U1: footprint (none) -> MacroLib:DIP-16
- U2: footprint (none) -> MacroLib:DIP-14
- U3: footprint (none) -> MacroLib:TO-220-3_Vertical
- U4: footprint (none) -> MacroLib:DIP-8
Connections:
- net GND: now also J5.1 (P1); no longer J5.3 (P3)
- net VCC: now also J5.3 (P3); no longer J5.1 (P1)
- net at R5.2, R8.2, U2.9 (-): now also J1.2; no longer J1.1
- net at D1.2 (K), D3.2 (K), R12.1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: now also R7.1
- net at R2.1, U2.1 (Out1): now also J1.1; no longer J1.2
Other:
- moved on the sheet: J1
