File: proyecto y diseño electornico/medidor de conductividad/medidor de conductividad.kicad_pcb (KiCad board)
At the start: 2 copper layers, 52 x 73 mm, 44 parts, among them J1 HEADER_2, J2 Cable_PAD, J3 Cable_PAD, J4 Cable_PAD, J5 CONN_01X03, U1 CD4060BM, U2 TL084, U3 LM317, U4 TC7660

Commit message: 10/5
Parts:
- moved R3 1.57 mm to (207.4, 49.0)
- moved C7 0.55 mm to (221.2, 83.2)
Routing:
- net Net-(J1-Pad1): track 48.8 -> 52.0 mm
- net Net-(R3-Pad2): track 40.1 -> 38.5 mm
- net GND: track 87.2 -> 85.9 mm
- net Net-(R2-Pad2): track 11.0 -> 12.2 mm
- net Net-(R11-Pad1): track 15.3 -> 14.8 mm
