File: proyecto y diseño electornico/distorder/distorder.kicad_sch (KiCad schematic)
At the start: 19 parts, among them J1 pw-, J2 pw+, J3 Out+, J4 In+, J5 Switch Mid, J6 Switch, J7 Switch, J8 Out-, J9 In-, Q1 BC546

Commit message: 1/11
Parts:
- C1: footprint (none) -> EESTN5:CAP_ELEC_8x11.5mm
- C2: footprint (none) -> EESTN5:CAP_0.1
- C3, C5: renamed from C?; footprint (none) -> EESTN5:CAP_0.1
- C4: renamed from C3; footprint (none) -> EESTN5:CAP_0.1
- D1: footprint (none) -> EESTN5:DO-41
- J1, J2, J3, J4, J5, J6, J7, J8, J9: footprint (none) -> EESTN5:Cable_Doble_1,5mm
- Q1: footprint EESTN5:TO-92 -> EESTN5:to92
- R1, R2, R3: footprint (none) -> EESTN5:RES0.2
