File: proyecto y diseño electornico/preamp/preamp.kicad_sch (KiCad schematic)
At the start: 0 parts

Commit message: 2/12
Parts:
- added C1: 10u, EESTN5:CAP_0.2, symbol EESTN5:C
- added C2: 10n, EESTN5:CAP_0.2, symbol EESTN5:C
- added C3: 1000u, EESTN5:CAP_ELEC_10X8mm, symbol EESTN5:C
- added C4: 22u, EESTN5:CAP_ELEC_5x11mm, symbol EESTN5:C
- added J1, J2, J3, J4: Cable_PAD, EESTN5:Cable_Doble_1,5mm, symbol EESTN5:Cable_PAD
- added R1, R2, R5: 10k, EESTN5:RES0.3, symbol EESTN5:R
- added R3: 1M, EESTN5:RES0.3, symbol EESTN5:R
- added R4: 5.1k, EESTN5:RES0.3, symbol EESTN5:R
- added U1: LM324, MacroLib:DIP-14, symbol macrolib:LM324
Connections:
- new net: C2.1, R3.2, U1.3 (+)
- new net: R4.1, U1.1, U1.2 (-)
- new net: R4.2, R5.1, U1.6 (-)
- new net: C4.1, R5.2, U1.7
- new net: C2.2, J1.1
- new net: C4.2, J4.1
- new net GND: C1.2, C3.1, J2.1, R2.1, R3.1, U1.10 (+), U1.11 (V-), U1.12 (+), U1.13 (-), U1.9 (-)
- new net VCC: C3.2, J3.1, R1.2, U1.4 (V+)
- new net virt_gnd: C1.1, R1.1, R2.2, U1.5 (+)
